File: mcu.kicad_sch (KiCad schematic)
At the start: 53 parts, among them J10 PinHeader_2x10_P1.27mm_SMD_Sh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, SW5 SW_B3U-1000P_SMD, SW6 CAS-120TA, U1 STM32H753ZIT6, Y1 Resonator_32.768kHz_ECX-31B, Y2 Oscillator_25MHz_ESC_2016MV

Commit message: [#95036] Connect remaining pins to MCU
Connections:
- net ACC_GYRO_INT1: now also U1.88 (PG3)
- net ACC_GYRO_INT2: now also U1.89 (PG4)
- net EN_PMOD: now also U1.113 (PC12)
- net EN_RPI_CONN: now also U1.48 (PB2)
- net GPIO0: now also U1.141 (PE0)
- net GPIO1: now also U1.142 (PE1)
- net GPIO16: now also U1.63 (PE10)
- net GPIO17: now also U1.65 (PE12)
- net GPIO20: now also U1.68 (PE15)
- net GPIO21: now also U1.13 (PF3)
- net GPIO22: now also U1.14 (PF4)
- net GPIO23: now also U1.15 (PF5)
- net GPIO24: now also U1.50 (PF12)
- net GPIO25: now also U1.56 (PG0)
- net GPIO26: now also U1.57 (PG1)
- net GPIO27: now also U1.87 (PG2)
- net GPIO5: now also U1.58 (PE7)
- net GPIO6: now also U1.59 (PE8)
- net MAG_~{INT}: now also U1.126 (PG11)
- net USB_GPIO_OUT1: now also U1.122 (PD6)
- net USB_GPIO_OUT2: now also U1.79 (PD10)
- net USB_GPIO_~{INT}: now also U1.116 (PD2)
- net ~{FTDI_RESET}: now also U1.7 (PC13)
Other:
- note removed: "33"
