File: can.kicad_sch (KiCad schematic)
At the start: 27 parts, among them J11 PinHeader_2x3_P2.54mm_Drill1.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, J12 PinHeader_1x2_P2.54mm_Drill1.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, J13 PinHeader_1x2_P2.54mm_Drill1.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, U19 TCAN3414DR, U20 TCAN3414DR

Commit message: [#95398] Cleanup
Parts:
- removed D19, D21: ESD2CAN24DCKRQ1, antmicro-footprints:SC70-3, symbol antmicroTVSDiodes:ESD2CAN24DCKRQ1
- removed J11: PinHeader_2x3_P2.54mm_Drill1.1mm, antmicro-footprints:PinHeader_2x3_P2.54mm_Drill1.1mm, symbol antmicroGenericPinHeaders:PinHeader_2x3_P2.54mm_Drill1.1mm
- removed J12, J13: PinHeader_1x2_P2.54mm_Drill1.1mm, antmicro-footprints:PinHeader_1x2_P2.54_Drill1.1mm, symbol antmicroGenericPinHeaders:PinHeader_1x2_P2.54mm_Drill1.1mm
- removed JP1, JP2: Jumper_1x2_P2.54mm, antmicro-footprints:Jumper_1x2_P2.54mm, symbol antmicroShuntsJumpers:Jumper_1x2_P2.54mm
- added R7: R_0R_0402, antmicro-footprints:R_0402_1005Metric, symbol antmicroResistors0402:R_0R_0402
- added SW7: CVS-03B, antmicro-footprints:SW_DIP_SPSTx03_Slide_Copal_CVS-03xB_W5.9mm_P1mm, symbol antmicroSlideSwitches:CVS-03B
Connections:
- net CAN1_H: now also SW7.5, SW7.6
- net CAN1_L: now also R7.1
- net CAN2_H: now also SW7.2, SW7.3
- net CAN2_L: now also R7.2
- net GND: now also SW7.7
- net CAN2_TERM: now reaches R161.2
- net CAN2_TERM: now also SW7.4
- net CAN1_TERM: now reaches R156.2
- net CAN1_TERM: now also SW7.1
Other:
- note added: "CAN Termination"
- note added: "SW7 legend: CAN1 Termination Loopback CAN2 Termination"
- moved on the sheet: C92, C93, C94, C95, C96, C97, R152, R153, R154, R155, R156, R157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

Commit message: [#95398] Schematic cleanup
Other:
- moved on the sheet: C92, C93, C94, C95, C96, C97, R152, R153, R154, R155, R156, R157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

Commit message: [#95398] Add markings for ETH strap resistors
Other:
- title: renode-reference-platform -> STM32H7 Renode Reference Platform
Changed lines of the file:
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@@
 	(paper "A3")
 	(title_block
-		(title "renode-reference-platform")
+		(title "STM32H7 Renode Reference Platform")
 		(date "07.04.2026")
 		(rev "1.0.0")
