File: can.kicad_sch (KiCad schematic)
At the start: 26 parts, among them J5 Wago_2059_1x3_2059-303/998-403, J6 Wago_2059_1x3_2059-303/998-403, U19 TCAN3414DR, U20 TCAN3414DR, U22 TS3A4751_X2QFN, U8 TS3A4751_X2QFN

Commit message: [#96159] Start PCB layout
Parts:
- added D19, D7: ESD2CAN24DBZRQ1, antmicro-footprints:SC70-3, symbol antmicroTVSDiodes:ESD2CAN24DBZRQ1
Connections:
- net GND: now also D19.3, D7.3
- net CAN1_H renamed CAN1+
- net CAN1+: now also J5.3, J5.4, D7.2; no longer J5.1, J5.2
- net CAN1_L renamed CAN1-
- net CAN1-: now also J5.1, J5.2, D7.1; no longer J5.3, J5.4
- net CAN2_H renamed CAN2+
- net CAN2+: now also J6.3, J6.4, D19.2; no longer J6.1, J6.2
- net CAN2_L renamed CAN2-
- net CAN2-: now also J6.1, J6.2, D19.1; no longer J6.3, J6.4
