File: can.kicad_sch (KiCad schematic)
At the start: 28 parts, among them J5 Wago_2059_1x3_2059-303/998-403, J6 Wago_2059_1x3_2059-303/998-403, U19 TCAN3414DR, U20 TCAN3414DR, U22 TS3A4751_X2QFN, U8 TS3A4751_X2QFN

Commit message: [#98579] Clean ERC
Parts:
- removed J5, J6: Wago_2059_1x3_2059-303/998-403, antmicro-footprints:WAGO_2059_1x3_2059-303-998-403, symbol Wire2BoardConnectors:WAGO_2059_1x3_2059-303-998-403
- added J5, J6: Wago_2059_1x3_2059-303/998-403, antmicro-footprints:WAGO_2059_1x3_2059-303-998-403, symbol antmicroWire2BoardConnectors:WAGO_2059_1x3_2059-303-998-403
Connections:
- net CAN1+: now also J5.3, J5.4
- net CAN1-: now also J5.1, J5.2
- net CAN2+: now also J6.3, J6.4
- net CAN2-: now also J6.1, J6.2
- net GND: now also J5.5, J5.6, J6.5, J6.6
