File: expansion.kicad_sch (KiCad schematic)
At the start: 6 parts, among them J8 JST_SH_1x4_SM04B-SRSS-TB-LF-SN

Commit message: [#95398] Add markings for ETH strap resistors
Other:
- title: renode-reference-platform -> STM32H7 Renode Reference Platform
Changed lines of the file:
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@@
 	(paper "A3")
 	(title_block
-		(title "renode-reference-platform")
+		(title "STM32H7 Renode Reference Platform")
 		(date "07.04.2026")
 		(rev "1.0.0")

Commit message: [#95451] Finalizing final placement
Other:
- note added: "I2C connector"
- note removed: "QWIIC"
Changed lines of the file:
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@@
 		(company "Antmicro")
 	)
-	(text "QWIIC\n"
+	(text "I2C connector"
 		(exclude_from_sim no)
 		(at 187.198 110.236 0)
