File: eth.kicad_sch (KiCad schematic)
At the start: 35 parts, among them J3 RJ45_Abracon_ARJM11B1-502-AB-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, U10 LAN8742A-CZ-TR, U9 TPD4E05U06QDQARQ1, Y3 Oscillator_25MHz_ESC_2016MV

Commit message: [#96159] Start PCB layout
Parts:
- added R41, R42, R44, R45, R46: R_0R_0402, antmicro-footprints:R_0402_1005Metric, symbol antmicroResistors0402:R_0R_0402
- added R60: R_33R_0402, antmicro-footprints:R_0402_1005Metric, symbol antmicroResistors0402:R_33R_0402
- added R63, R65: R_10k_0402, antmicro-footprints:R_0402_1005Metric, symbol antmicroResistors0402:R_10k_0402
Connections:
- net +3V3: now also C27.2, U10.9 (VDDIO)
- net 3V3_ETH: no longer C27.2, U10.9 (VDDIO)
- net GND: now also R63.1, R65.1
- net LED1: now also R63.2
- net LED2: now also R65.2
- net RMII.MDC: now also R41.1; no longer U10.13 (MDC)
- net RMII.MDIO: now also R42.1; no longer R35.1, U10.12 (MDIO)
- net RMII.REF_CLK: now also R60.1; no longer R31.1, U10.14 (~{INT})
- net RMII.TXD0: now also R44.1; no longer U10.17 (TXD0)
- net RMII.TXD1: now also R46.1; no longer U10.18 (TXD1)
- net RMII.TX_EN: now also R45.1; no longer U10.16 (TXEN)
- net RXN: now also U9.4, U9.7; no longer U9.5, U9.6
- net RXP: now also U9.5, U9.6; no longer U9.4, U9.7
- net TXN: now also U9.1, U9.10; no longer U9.2, U9.9
- net TXP: now also U9.2, U9.9; no longer U9.1, U9.10
- new net: R35.1, R42.2, U10.12 (MDIO)
- new net: R31.1, R60.2, U10.14 (~{INT})
- new net: R46.2, U10.18 (TXD1)
- new net: R41.2, U10.13 (MDC)
- new net: R45.2, U10.16 (TXEN)
- new net: R44.2, U10.17 (TXD0)
Other:
- moved on the sheet: C27, C28, C32, R25, R36, Y3
