File: usb-c.kicad_sch (KiCad schematic)
At the start: 40 parts, among them J2 USB-C_GCT_USB4105-GF-A, U12 FUSB303B, U13 AP22615B_TSOT26

Commit message: [#95398] Cleanup
Parts:
- R98: now fitted
Changed lines of the file:
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@@
 		(in_bom yes)
 		(on_board yes)
-		(dnp yes)
+		(dnp no)
 		(fields_autoplaced yes)
 		(property "Reference" "R98"

Commit message: [#95398] Implement basic post review sugestions
Parts:
- removed R102, R103: R_100R_0402, antmicro-footprints:R_0402_1005Metric, symbol antmicroResistors0402:R_100R_0402
Connections:
- net USB.D+: now also J2.A6 (D_{A}+), J2.B6 (D_{B}+)
- net USB.D-: now also J2.A7 (D_{A}-), J2.B7 (D_{B}-)

Commit message: [#95398] Add markings for ETH strap resistors
Other:
- title: renode-reference-platform -> STM32H7 Renode Reference Platform
Changed lines of the file:
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@@
 	(paper "A3")
 	(title_block
-		(title "renode-reference-platform")
+		(title "STM32H7 Renode Reference Platform")
 		(date "07.04.2026")
 		(rev "1.0.0")

Commit message: [#95451] Finalizing final placement
Parts:
- removed R79: R_0R_0402, antmicro-footprints:R_0402_1005Metric, symbol antmicroResistors0402:R_0R_0402
Changed lines of the file:
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@@
 	(wire
 		(pts
-			(xy 116.84 105.41) (xy 132.08 105.41)
+			(xy 121.92 105.41) (xy 140.97 105.41)
 		)
 		(stroke
@@
 	(wire
 		(pts
-			(xy 137.16 105.41) (xy 140.97 105.41)
-		)
-		(stroke
-			(width 0)
-			(type default)
-		)
-	)
-	(wire
-		(pts
 			(xy 205.74 137.16) (xy 210.82 137.16)
 		)
@@
 	(wire
 		(pts
-			(xy 205.74 132.08) (xy 205.74 121.92)
+			(xy 207.01 132.08) (xy 207.01 121.92)
 		)
 		(stroke
@@
 	(wire
 		(pts
+			(xy 207.01 132.08) (xy 205.74 132.08)
+		)
+		(stroke
+			(width 0)
+			(type default)
+		)
+	)
+	(wire
+		(pts
 			(xy 256.54 107.95) (xy 251.46 107.95)
 		)
@@
 	(wire
 		(pts
-			(xy 205.74 121.92) (xy 210.82 121.92)
+			(xy 207.01 121.92) (xy 210.82 121.92)
 		)
 		(stroke
@@
 	)
 	(label "USB.VBUS"
-		(at 116.84 105.41 0)
+		(at 121.92 105.41 0)
 		(effects
 			(font
@@
 					(unit 1)
 				)
-			)
-		)
-	)
-	(symbol
-		(lib_id "antmicroResistors0402:R_0R_0402")
-		(at 132.08 105.41 0)
-		(unit 1)
-		(exclude_from_sim no)
-		(in_bom yes)
-		(on_board yes)
-		(dnp no)
-		(fields_autoplaced yes)
-		(property "Reference" "R79"
-			(at 134.62 99.06 0)
-			(effects
-				(font
-					(size 1.27 1.27)
-					(thickness 0.15)
-				)
-			)
-		)
-		(property "Value" "R_0R_0402"
-			(at 152.4 118.11 0)
-			(effects
-				(font
-					(size 1.27 1.27)
-					(thickness 0.15)
-				)
-				(justify left bottom)
-				(hide yes)
-			)
-		)
-		(property "Footprint" "antmicro-footprints:R_0402_1005Metric"
-			(at 152.4 120.65 0)
-			(effects
-				(font
-					(size 1.27 1.27)
-					(thickness 0.15)
-				)
-				(justify left bottom)
-				(hide yes)
-			)
-		)
-		(property "Datasheet" "https://industrial.panasonic.com/cdbs/www-data/pdf/RDA0000/AOA0000C301.pdf"
-			(at 152.4 123.19 0)
-			(effects
-				(font
-					(size 1.27 1.27)
-					(thickness 0.15)
-				)
-				(justify left bottom)
-				(hide yes)
-			)
-		)
-		(property "Description" "SMD Chip Resistor, Jumper, 0 ohm, 100 mW, 0402 [1005 Metric], Thick Film, General Purpose"
-			(at 152.4 138.43 0)
-			(effects
-				(font
-					(size 1.27 1.27)
-				)
-				(justify left bottom)
-				(hide yes)
-			)
-		)
-		(property "MPN" "ERJ2GE0R00X"
-			(at 152.4 125.73 0)
-			(effects
-				(font
-					(size 1.27 1.27)
-					(thickness 0.15)
-				)
-				(justify left bottom)
-				(hide yes)
-			)
-		)
-		(property "Manufacturer" "Panasonic"
-			(at 152.4 128.27 0)
-			(effects
-				(font
-					(size 1.27 1.27)
-					(thickness 0.15)
-				)
-				(justify left bottom)
-				(hide yes)
-			)
-		)
-		(property "License" "Apache-2.0"
-			(at 152.4 130.81 0)
-			(effects
-				(font
-					(size 1.27 1.27)
-					(thickness 0.15)
-				)
-				(justify left bottom)
-				(hide yes)
-			)
-		)
-		(property "Author" "Antmicro"
-			(at 152.4 133.35 0)
-			(effects
-				(font
-					(size 1.27 1.27)
-					(thickness 0.15)
-				)
-				(justify left bottom)
-				(hide yes)
-			)
-		)
-		(property "Val" "0R"
-			(at 134.62 101.6 0)
-			(effects
-				(font
-					(size 1.27 1.27)
-					(thickness 0.15)
-				)
-			)
-		)
-		(property "Tolerance" "~"
-			(at 152.4 115.57 0)
-			(effects
-				(font
-					(size 1.27 1.27)
-				)
-				(justify left bottom)
-				(hide yes)
-			)
-		)
-		(property "Current" "1A"
-			(at 152.4 135.89 0)
-			(effects
-				(font
-					(size 1.27 1.27)
-					(thickness 0.15)
-				)
-				(justify left bottom)
-				(hide yes)
-			)
-		)
-		(pin "1"
-		)
-		(pin "2"
-		)
-		(instances
-			(project "renode-reference-platform"
-				(path "/126ae87b-f292-4372-94ff-ae46971d67ab/ec770658-59a1-4a3f-81ed-5fcccc21c2e8"
-					(reference "R79")
-					(unit 1)
-				)

Commit message: [#96159] Continue PCB layout
Connections:
- net CC1: now also D11.2; no longer D11.1
- net CC2: now also D11.1; no longer D11.2
- net USB.D+: now also D8.2; no longer D8.1
- net USB.D-: now also D8.1; no longer D8.2
Changed lines of the file:
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@@
 	)
 	(label "USB.D-"
-		(at 130.81 189.23 0)
+		(at 130.81 186.69 0)
 		(effects
 			(font
@@
 	)
 	(label "CC1"
-		(at 167.64 186.69 0)
+		(at 167.64 189.23 0)
 		(effects
 			(font
@@
 	)
 	(label "USB.D+"
-		(at 130.81 186.69 0)
+		(at 130.81 189.23 0)
 		(effects
 			(font
@@
 	)
 	(label "CC2"
-		(at 167.64 189.23 0)
+		(at 167.64 186.69 0)
 		(effects
 			(font

Commit message: [#96159] Power and low speed layout
Connections:
- net USB.D+: now also D8.1; no longer D8.2
- net USB.D-: now also D8.2; no longer D8.1
Changed lines of the file:
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@@
 	)
 	(label "USB.D-"
-		(at 130.81 186.69 0)
+		(at 130.81 189.23 0)
 		(effects
 			(font
@@
 	)
 	(label "USB.D+"
-		(at 130.81 189.23 0)
+		(at 130.81 186.69 0)
 		(effects
 			(font
@@
 		)
 	)
+	(rule_area
+		(polyline
+			(pts
+				(xy 129.54 143.51) (xy 135.89 143.51) (xy 135.89 151.13) (xy 129.54 151.13)
+			)
+			(stroke
+				(width 0)
+				(type dash)
+			)
+			(fill
+				(type none)
+			)
+		)
+	)
+	(netclass_flag ""
+		(length 2.54)
+		(shape round)
+		(at 129.54 151.13 180)
+		(fields_autoplaced yes)
+		(effects
+			(font
+				(size 1.27 1.27)
+			)
+			(justify right bottom)
+		)
+		(property "Netclass" "90Ohm-diff_USB"
+			(at 130.2385 153.67 0)
+			(effects
+				(font
+					(size 1.27 1.27)
+				)
+				(justify left)
+			)
+		)
+		(property "Component Class" ""
+			(at -64.77 15.24 0)
+			(effects
+				(font
+					(size 1.27 1.27)
+					(italic yes)
+				)
+			)
+		)
+	)
