File: imu.kicad_sch (KiCad schematic)
At the start: 24 parts, among them U3 IIS2MDCTR, U4 LSM6DSO32TR, U5 TMP108AIYFFR, U6 LPS25HBTR, U8 OPT4001DTSR

Commit message: Rename project
Other:
- title: renode-reference-platform -> stm32h7-renode-reference-platform
