File: pmod.kicad_sch (KiCad schematic)
At the start: 14 parts, among them J5 PinSocket_2x6_P2.54mm_Drill1.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, J6 PinSocket_2x6_P2.54mm_Drill1.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, U11 NCP380LSNAJAAT1G

Commit message: Rename project
Other:
- title: renode-reference-platform -> stm32h7-renode-reference-platform
Changed lines of the file:
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@@
 	(paper "A3")
 	(title_block
-		(title "renode-reference-platform")
+		(title "stm32h7-renode-reference-platform")
 		(date "07.04.2026")
 		(rev "1.0.0")
@@
 		)
 		(instances
-			(project "renode-reference-platform"
+			(project "stm32h7-renode-reference-platform"
 				(path "/126ae87b-f292-4372-94ff-ae46971d67ab/8150c4f5-86f0-4781-bc9c-6f93770faa9d"
 					(reference "R50")
@@
 		)
 		(instances
-			(project "renode-reference-platform"
+			(project "stm32h7-renode-reference-platform"
 				(path "/126ae87b-f292-4372-94ff-ae46971d67ab/8150c4f5-86f0-4781-bc9c-6f93770faa9d"
 					(reference "D23")
@@
 		)
 		(instances
-			(project "renode-reference-platform"
+			(project "stm32h7-renode-reference-platform"
 				(path "/126ae87b-f292-4372-94ff-ae46971d67ab/8150c4f5-86f0-4781-bc9c-6f93770faa9d"
 					(reference "D26")
@@
 		)
 		(instances
-			(project "renode-reference-platform"
+			(project "stm32h7-renode-reference-platform"
 				(path "/126ae87b-f292-4372-94ff-ae46971d67ab/8150c4f5-86f0-4781-bc9c-6f93770faa9d"
 					(reference "R47")
@@
 		)
 		(instances
-			(project "renode-reference-platform"
+			(project "stm32h7-renode-reference-platform"
 				(path "/126ae87b-f292-4372-94ff-ae46971d67ab/8150c4f5-86f0-4781-bc9c-6f93770faa9d"
 					(reference "#PWR066")
@@
 		)
 		(instances
-			(project "renode-reference-platform"
+			(project "stm32h7-renode-reference-platform"
 				(path "/126ae87b-f292-4372-94ff-ae46971d67ab/8150c4f5-86f0-4781-bc9c-6f93770faa9d"
 					(reference "J5")
@@
 		)
 		(instances
-			(project "renode-reference-platform"
+			(project "stm32h7-renode-reference-platform"
 				(path "/126ae87b-f292-4372-94ff-ae46971d67ab/8150c4f5-86f0-4781-bc9c-6f93770faa9d"
 					(reference "#PWR064")
@@
 		)
 		(instances
-			(project "renode-reference-platform"
+			(project "stm32h7-renode-reference-platform"
 				(path "/126ae87b-f292-4372-94ff-ae46971d67ab/8150c4f5-86f0-4781-bc9c-6f93770faa9d"
 					(reference "#PWR065")
@@
 		)
 		(instances
-			(project "renode-reference-platform"
+			(project "stm32h7-renode-reference-platform"
 				(path "/126ae87b-f292-4372-94ff-ae46971d67ab/8150c4f5-86f0-4781-bc9c-6f93770faa9d"
 					(reference "C36")
@@
 		)
 		(instances
-			(project "renode-reference-platform"
+			(project "stm32h7-renode-reference-platform"
 				(path "/126ae87b-f292-4372-94ff-ae46971d67ab/8150c4f5-86f0-4781-bc9c-6f93770faa9d"
 					(reference "#PWR0214")
@@
 		)
 		(instances
-			(project "renode-reference-platform"
+			(project "stm32h7-renode-reference-platform"
 				(path "/126ae87b-f292-4372-94ff-ae46971d67ab/8150c4f5-86f0-4781-bc9c-6f93770faa9d"
 					(reference "J6")
@@
 		)
 		(instances
-			(project "renode-reference-platform"
+			(project "stm32h7-renode-reference-platform"
 				(path "/126ae87b-f292-4372-94ff-ae46971d67ab/8150c4f5-86f0-4781-bc9c-6f93770faa9d"
 					(reference "C37")
@@
 		)
 		(instances
-			(project "renode-reference-platform"
+			(project "stm32h7-renode-reference-platform"
 				(path "/126ae87b-f292-4372-94ff-ae46971d67ab/8150c4f5-86f0-4781-bc9c-6f93770faa9d"
 					(reference "D25")
@@
 		)
 		(instances
-			(project "renode-reference-platform"
+			(project "stm32h7-renode-reference-platform"
 				(path "/126ae87b-f292-4372-94ff-ae46971d67ab/8150c4f5-86f0-4781-bc9c-6f93770faa9d"
 					(reference "#PWR063")
@@
 		)
 		(instances
-			(project "renode-reference-platform"
+			(project "stm32h7-renode-reference-platform"
 				(path "/126ae87b-f292-4372-94ff-ae46971d67ab/8150c4f5-86f0-4781-bc9c-6f93770faa9d"
 					(reference "D24")
@@
 		)
 		(instances
-			(project "renode-reference-platform"
+			(project "stm32h7-renode-reference-platform"
 				(path "/126ae87b-f292-4372-94ff-ae46971d67ab/8150c4f5-86f0-4781-bc9c-6f93770faa9d"
 					(reference "R48")
@@
 		)
 		(instances
-			(project "renode-reference-platform"
+			(project "stm32h7-renode-reference-platform"
 				(path "/126ae87b-f292-4372-94ff-ae46971d67ab/8150c4f5-86f0-4781-bc9c-6f93770faa9d"
 					(reference "#PWR059")
@@
 		)
 		(instances
-			(project "renode-reference-platform"
+			(project "stm32h7-renode-reference-platform"
 				(path "/126ae87b-f292-4372-94ff-ae46971d67ab/8150c4f5-86f0-4781-bc9c-6f93770faa9d"
 					(reference "#PWR061")
@@
 		)
 		(instances
-			(project "renode-reference-platform"
+			(project "stm32h7-renode-reference-platform"
 				(path "/126ae87b-f292-4372-94ff-ae46971d67ab/8150c4f5-86f0-4781-bc9c-6f93770faa9d"
 					(reference "#PWR060")
@@
 		)
 		(instances
-			(project "renode-reference-platform"
+			(project "stm32h7-renode-reference-platform"
 				(path "/126ae87b-f292-4372-94ff-ae46971d67ab/8150c4f5-86f0-4781-bc9c-6f93770faa9d"
 					(reference "#PWR062")
@@
 		)
 		(instances
-			(project "renode-reference-platform"
+			(project "stm32h7-renode-reference-platform"
 				(path "/126ae87b-f292-4372-94ff-ae46971d67ab/8150c4f5-86f0-4781-bc9c-6f93770faa9d"
 					(reference "#PWR0213")
@@
 		)
 		(instances
-			(project "renode-reference-platform"
+			(project "stm32h7-renode-reference-platform"
 				(path "/126ae87b-f292-4372-94ff-ae46971d67ab/8150c4f5-86f0-4781-bc9c-6f93770faa9d"
 					(reference "#PWR0122")
@@
 		)
 		(instances
-			(project "renode-reference-platform"
+			(project "stm32h7-renode-reference-platform"
 				(path "/126ae87b-f292-4372-94ff-ae46971d67ab/8150c4f5-86f0-4781-bc9c-6f93770faa9d"
 					(reference "U11")
@@
 		)
 		(instances
-			(project "renode-reference-platform"
+			(project "stm32h7-renode-reference-platform"
 				(path "/126ae87b-f292-4372-94ff-ae46971d67ab/8150c4f5-86f0-4781-bc9c-6f93770faa9d"
 					(reference "R49")
@@
 		)
 		(instances
-			(project "renode-reference-platform"
+			(project "stm32h7-renode-reference-platform"
 				(path "/126ae87b-f292-4372-94ff-ae46971d67ab/8150c4f5-86f0-4781-bc9c-6f93770faa9d"
 					(reference "#PWR0212")
@@
 		)
 		(instances
-			(project "renode-reference-platform"
+			(project "stm32h7-renode-reference-platform"
 				(path "/126ae87b-f292-4372-94ff-ae46971d67ab/8150c4f5-86f0-4781-bc9c-6f93770faa9d"
 					(reference "C35")
