File: rpi-expansion.kicad_sch (KiCad schematic)
At the start: 6 parts, among them J8 JST_SH_1x4_SM04B-SRSS-TB-LF-SN

Commit message: Rename project
Other:
- title: renode-reference-platform -> stm32h7-renode-reference-platform
Changed lines of the file:
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@@
 	(paper "A3")
 	(title_block
-		(title "renode-reference-platform")
+		(title "stm32h7-renode-reference-platform")
 		(date "07.04.2026")
 		(rev "1.0.0")
@@
 		)
 		(instances
-			(project "renode-reference-platform"
+			(project "stm32h7-renode-reference-platform"
 				(path "/126ae87b-f292-4372-94ff-ae46971d67ab/3deaa797-f1d6-4980-9fc1-21264c177bf0"
 					(reference "#PWR02")
@@
 		)
 		(instances
-			(project "renode-reference-platform"
+			(project "stm32h7-renode-reference-platform"
 				(path "/126ae87b-f292-4372-94ff-ae46971d67ab/3deaa797-f1d6-4980-9fc1-21264c177bf0"
 					(reference "#PWR0216")
@@
 		)
 		(instances
-			(project "renode-reference-platform"
+			(project "stm32h7-renode-reference-platform"
 				(path "/126ae87b-f292-4372-94ff-ae46971d67ab/3deaa797-f1d6-4980-9fc1-21264c177bf0"
 					(reference "R4")
@@
 		)
 		(instances
-			(project "renode-reference-platform"
+			(project "stm32h7-renode-reference-platform"
 				(path "/126ae87b-f292-4372-94ff-ae46971d67ab/3deaa797-f1d6-4980-9fc1-21264c177bf0"
 					(reference "D28")
@@
 		)
 		(instances
-			(project "renode-reference-platform"
+			(project "stm32h7-renode-reference-platform"
 				(path "/126ae87b-f292-4372-94ff-ae46971d67ab/3deaa797-f1d6-4980-9fc1-21264c177bf0"
 					(reference "R5")
@@
 		)
 		(instances
-			(project "renode-reference-platform"
+			(project "stm32h7-renode-reference-platform"
 				(path "/126ae87b-f292-4372-94ff-ae46971d67ab/3deaa797-f1d6-4980-9fc1-21264c177bf0"
 					(reference "#PWR04")
@@
 		)
 		(instances
-			(project "renode-reference-platform"
+			(project "stm32h7-renode-reference-platform"
 				(path "/126ae87b-f292-4372-94ff-ae46971d67ab/3deaa797-f1d6-4980-9fc1-21264c177bf0"
 					(reference "TP17")
@@
 		)
 		(instances
-			(project "renode-reference-platform"
+			(project "stm32h7-renode-reference-platform"
 				(path "/126ae87b-f292-4372-94ff-ae46971d67ab/3deaa797-f1d6-4980-9fc1-21264c177bf0"
 					(reference "#PWR03")
@@
 		)
 		(instances
-			(project "renode-reference-platform"
+			(project "stm32h7-renode-reference-platform"
 				(path "/126ae87b-f292-4372-94ff-ae46971d67ab/3deaa797-f1d6-4980-9fc1-21264c177bf0"
 					(reference "TP16")
@@
 		)
 		(instances
-			(project "renode-reference-platform"
+			(project "stm32h7-renode-reference-platform"
 				(path "/126ae87b-f292-4372-94ff-ae46971d67ab/3deaa797-f1d6-4980-9fc1-21264c177bf0"
 					(reference "J8")
