File: spi-flash.kicad_sch (KiCad schematic)
At the start: 19 parts, among them J4 Tag-Connect_TC2050-IDC-NL_2x5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, U14 MT25QL01GBBB8E_SOP2-16

Commit message: [#100413] Change QSPI-Flash to IS25LP01GJ-RMLE, Update pull-ups to FLASH_PWR rail
Parts:
- removed U14: MT25QL01GBBB8E_SOP2-16, antmicro-footprints:SOP2-16_7.5x10.3mm, symbol antmicroMemory:MT25QL01GBBB8E_SOP2-16
- added R346: R_10k_0402, antmicro-footprints:R_0402_1005Metric, symbol antmicroResistors0402:R_10k_0402
- added U14: IS25LP01GJ-RMLE, antmicro-footprints:SOP2-16_7.5x10.3mm, symbol antmicroMemory:IS25LP01GJ-RMLE
Connections:
- net +3V3: no longer R343.2, R344.2, R345.2
- net FLASH_CLK: now also U14.16 (SCK)
- net FLASH_IO2: now also U14.9 (~{WP})
- net FLASH_IO3: now also U14.1 (~{HOLD})
- net FLASH_MISO_IO1: now also U14.8 (SO)
- net FLASH_MOSI_IO0: now also U14.15 (SI)
- net FLASH_PWR: now also R343.2, R344.2, R345.2, R346.2, U14.2 (VCC)
- net FLASH_~{CS}: now also U14.7 (~{CE})
- net GND: now also U14.10 (GND)
- new net: U14.11 (NC), U14.12 (NC), U14.13 (NC), U14.14 (NC), U14.4 (NC), U14.5 (NC), U14.6 (NC)
- new net: R346.1, U14.3 (~{RESET})
- no-connect marks 2 -> 1
